Commit message: Add COBOTTA claw model and collision scene

File: src/dual_robot_description/urdf/dual_robot.urdf (robot description, URDF)
Before this commit: robot cobotta_mycobot_dual_robot, 18 links, 17 joints
Links:
- added link mycobot_tool_link; collision cylinder length=0.020 radius=0.014; visual cylinder length=0.020 radius=0.014
- link cobotta_left_finger: geometry collision mesh filename=package://dual_robot_description/meshes/cobotta/COBOTTA_gri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 scale=0.001 0.001 0.001; visual mesh filename=package://dual_robot_description/meshes/cobotta/COBOTTA_gri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 scale=0.001 0.001 0.001
- link cobotta_right_finger: geometry collision mesh filename=package://dual_robot_description/meshes/cobotta/COBOTTA_gri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 scale=0.001 0.001 0.001; visual mesh filename=package://dual_robot_description/meshes/cobotta/COBOTTA_gri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 scale=0.001 0.001 0.001
Joints:
- added joint mycobot_tool_fixed_joint: type fixed, parent mycobot_link6, child mycobot_tool_link, origin xyz=0 0 0 rpy=0 0 0
- joint cobotta_joint_w: origin xyz=0 0 0.025 rpy=0 0 0 -> xyz=0 0 0.022 rpy=0 0 0

Commit message: Validate COBOTTA position-only planning from Unity grasp point

File: src/dual_robot_description/urdf/dual_robot.urdf (robot description, URDF)
Before this commit: robot cobotta_mycobot_dual_robot, 19 links, 18 joints
Links:
- added link cobotta_tool_link; visual sphere radius=0.002
Joints:
- added joint cobotta_tool_joint: type fixed, parent cobotta_gripper_base, child cobotta_tool_link, origin xyz=-0.003 0 0.080 rpy=0 0 0

Commit message: Add Test7 robot tools mounts and integrated launch

File: src/dual_robot_description/urdf/dual_robot.urdf (robot description, URDF)
Before this commit: robot cobotta_mycobot_dual_robot, 20 links, 19 joints
Links:
- link mycobot_tool_link: geometry collision cylinder length=0.020 radius=0.014; visual cylinder length=0.002 radius=0.0085
Joints:
- joint cobotta_joint_gripper: origin xyz=0.000000 0.000000 0.06000 rpy=0.000000 0.000000 0.000000 -> xyz=0.000000 0.008750 0.06000 rpy=0.000000 0.000000 0.000000
- joint cobotta_joint_gripper_mimic: origin xyz=0.000000 0.000000 0.060000 rpy=0.000000 0.000000 0.000000 -> xyz=0.000000 -0.002250 0.060000 rpy=0.000000 0.000000 0.000000
- joint cobotta_tool_joint: origin xyz=-0.003 0 0.080 rpy=0 0 0 -> xyz=-0.002 0 0.080 rpy=0 0 0

Commit message: Add Test7 paper adjustment tool holders

File: src/dual_robot_description/urdf/dual_robot.urdf (robot description, URDF)
Before this commit: robot cobotta_mycobot_dual_robot, 20 links, 19 joints
Links:
- added link cap_case_link; visual mesh filename=package://dual_robot_description/meshes/environment/cap_cas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 scale=0.001 0.001 0.001
- added link hand_cap_link; visual mesh filename=package://dual_robot_description/meshes/environment/hand_ca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 scale=0.001 0.001 0.001
- added link set_tool_base_link; visual mesh filename=package://dual_robot_description/meshes/environment/set_too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 scale=0.001 0.001 0.001
Joints:
- added joint world_to_cap_case: type fixed, parent world, child cap_case_link, origin xyz=-0.0265 -0.130 0.120 rpy=1.5708 3.14159 0
- added joint world_to_hand_cap: type fixed, parent world, child hand_cap_link, origin xyz=-0.085 -0.160 0.030 rpy=0 0 0
- added joint world_to_set_tool_base: type fixed, parent world, child set_tool_base_link, origin xyz=0.025 -0.175 0.0495 rpy=1.5708 0 0

Commit message: Add Test7 tool and holder collision models

File: src/dual_robot_description/urdf/dual_robot.urdf (robot description, URDF)
Before this commit: robot cobotta_mycobot_dual_robot, 23 links, 22 joints
Links:
- link cap_case_link: geometry collision mesh filename=package://dual_robot_description/meshes/environment/cap_cas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 scale=0.001 0.001 0.001; visual mesh filename=package://dual_robot_description/meshes/environment/cap_cas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 scale=0.001 0.001 0.001
- link hand_cap_link: geometry collision mesh filename=package://dual_robot_description/meshes/environment/hand_ca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 scale=0.001 0.001 0.001; visual mesh filename=package://dual_robot_description/meshes/environment/hand_ca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 scale=0.001 0.001 0.001
- link mycobot_tool_link: geometry collision cylinder length=0.002 radius=0.0085; collision cylinder length=0.018 radius=0.006
- link set_tool_base_link: geometry collision mesh filename=package://dual_robot_description/meshes/environment/set_too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 scale=0.001 0.001 0.001; visual mesh filename=package://dual_robot_description/meshes/environment/set_too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 scale=0.001 0.001 0.001

Commit message: Add COBOTTA set cap tool model

File: src/dual_robot_description/urdf/dual_robot.urdf (robot description, URDF)
Before this commit: robot cobotta_mycobot_dual_robot, 23 links, 22 joints
Links:
- added link set_cap_link; collision mesh filename=package://dual_robot_description/meshes/cobotta/set_cap.stl scale=0.001 0.001 0.001; visual mesh filename=package://dual_robot_description/meshes/cobotta/set_cap.stl scale=0.001 0.001 0.001
Joints:
- added joint set_tool_base_to_set_cap: type fixed, parent set_tool_base_link, child set_cap_link, origin xyz=0.000 -0.09196 -0.00018 rpy=-1.5708 0 0

Commit message: Add MyCobot contact boundary and folded paper collision tools

File: src/dual_robot_description/urdf/dual_robot.urdf (robot description, URDF)
Before this commit: robot cobotta_mycobot_dual_robot, 24 links, 23 joints
Links:
- added link mycobot_crease_tcp
Joints:
- added joint mycobot_crease_tcp_joint: type fixed, parent mycobot_tool_link, child mycobot_crease_tcp, origin xyz=0.0053 -0.001 0.0373 rpy=0 0 0

Commit message: Add MyCobot allowed contact region and collision diagnostics

File: src/dual_robot_description/urdf/dual_robot.urdf (robot description, URDF)
Before this commit: robot cobotta_mycobot_dual_robot, 25 links, 24 joints
Links:
- added link mycobot_allowed_contact_link; collision mesh filename=package://dual_robot_description/meshes/mycobot/tool/mycobo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 scale=0.001 0.001 0.001; visual mesh filename=package://dual_robot_description/meshes/mycobot/tool/mycobo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 scale=0.001 0.001 0.001
Joints:
- added joint mycobot_allowed_contact_joint: type fixed, parent mycobot_tool_link, child mycobot_allowed_contact_link, origin xyz=0 0 0 rpy=0 0 0
